File: hardware/keypad.kicad_sch (KiCad schematic)
At the start: 49 parts, among them SW1 TRIG1, SW10 TRIG10, SW11 TRIG11, SW12 TRIG12, SW13 TRIG13, SW14 TRIG14, SW15 TRIG15, SW16 TRIG16, SW2 TRIG2, SW3 TRIG3, SW4 TRIG4, SW5 TRIG5, SW6 TRIG6, SW7 TRIG7, SW8 TRIG8, SW9 TRIG9, U10 TRIG9, U11 TRIG13, U12 TRIG10, U13 TRIG14, U14 TRIG11, U15 TRIG15, U16 TRIG12, U17 TRIG16, U2 TRIG1, U25 TCA8418RTWR, U3 TRIG2, U4 TRIG3, U5 TRIG4, U6 TRIG8, U7 TRIG7, U8 TRIG6, U9 TRIG5

Commit message: feat: various layout adjustments
Other:
- note added: "TODO: op-amp based level converter, see adafruit neokey projects"
Changed lines of the file:
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@@
 	(generator_version "9.0")
 	(paper "A4")
+	(text "TODO: op-amp based level converter,\nsee adafruit neokey projects"
+		(exclude_from_sim no)
+		(at 176.784 41.148 0)
+		(effects
+			(font
+				(size 1.27 1.27)
+				(thickness 0.254)
+				(bold yes)
+				(color 194 0 0 1)
+			)
+		)
+	)
 	(junction
 		(at 34.29 26.67)
