File: hardware/pocket_synth.kicad_pcb (KiCad board)
At the start: 4 copper layers, 72 x 150 mm, 96 parts, among them J10 MIDI_OUT, J2 USB, J3 Micro_SD_Card_Det_Hirose_DM3AT, J6 LINE_IN, J8 LINE_OUT, J9 MIDI_IN, SW1 TRIG1, SW10 TRIG10, SW11 TRIG11, SW12 TRIG12, SW13 TRIG13, SW14 TRIG14, SW15 TRIG15, SW16 TRIG16, SW2 TRIG2, SW3 TRIG3, SW4 TRIG4, SW5 TRIG5, SW6 TRIG6, SW7 TRIG7, SW8 TRIG8, SW9 TRIG9, U1 VOL_PWR_POT, U10 TRIG9, U11 TRIG13, U12 TRIG10, U13 TRIG14, U14 TRIG11, U15 TRIG15, U16 TRIG12, U17 TRIG16, U18 STM32H743ZIT6, U2 TRIG1, U20 TPS62A02DRL, U21 TPS560200, U24 STM6601, U25 TCA8418RTWR, U3 TRIG2, U4 TRIG3, U5 TRIG4, U6 TRIG8, U7 TRIG7, U8 TRIG6, U9 TRIG5

Commit message: feat: various layout adjustments
Parts:
- removed TP16: SYS, TestPoint:TestPoint_Pad_D1.0mm
- removed U24: STM6601, Package_DFN_QFN:TDFN-12_2x3mm_P0.5mm
- added U22: MAX17261xxTD, Package_DFN_QFN:TDFN-14-1EP_3x3mm_P0.4mm_EP1.78x2.35mm, F.Cu at (-48.8, 144.7)
- added U23: BQ21040DBV, Package_TO_SOT_SMD:SOT-23-6, F.Cu at (-43.6, 144.6)
- added U26: FUSB303BTMX, Package_DFN_QFN:Texas_X2QFN-12_1.6x1.6mm_P0.4mm, F.Cu at (-35.4, 133.0)
- added U27: FUSB302B01MPX, Package_DFN_QFN:WQFN-14-1EP_2.5x2.5mm_P0.5mm_EP1.45x1.45mm, F.Cu at (-38.7, 144.5)
- D17: value POWER -> PWR
- U1: moved to F.Cu
- moved U1 9.36 mm to (46.8, 51.0)
- moved U19 6.50 mm to (79.2, 68.9)
- moved D17 4.11 mm to (63.3, 36.1), turned to -90 degrees
Connections:
- net /Power/3v3_EN renamed /Power/~{PWR_EN}
- C50 pad 1: /Power/SYS -> VDD
- D17 pad 1: unconnected-(D17-K-Pad1) -> Net-(D17-K)
- D17 pad 2: unconnected-(D17-A-Pad2) -> +3.3V
- U1 pad 4: unconnected-(U1-SW-Pad4) -> VDD
- U1 pad 5: unconnected-(U1-SW-Pad5) -> /Power/MCU_PWR_SW
- U20 pad 3: /Power/SYS -> VDD
Other:
- outline, holes or cut-outs redrawn
