File: hardware/power.kicad_sch (KiCad schematic)
At the start: 30 parts, among them J2 USB, U1 VOL_PWR_POT, U20 TPS62A02DRL, U21 TPS560200, U22 MAX17261xxTD, U23 BQ21040DBV, U26 FUSB303BTMX, U27 FUSB302B01MPX

Commit message: feat: various layout adjustments
Parts:
- added D19: D, symbol Device:D
- added R3: 10k, symbol Device:R
Connections:
- net +3.3V: now also D17.2 (A)
- net GND: now also R3.2; no longer R2.2
- net PWR_EN renamed ~{PWR_EN}
- net ~{PWR_EN}: now also D19.1 (K); no longer D17.2 (A)
- new net ~{MCU_PWR_EN}: D19.2 (A), R3.1
Other:
- note added: "3.3v GPIO-based soft power off enable"
- note added: "3.6-5.2v battery/charge voltage"
- note added: "EN logic high = 1.2v"
- note added: "Soft power-off is enabled by latching the power on with GPIO once the MCU has booted, and only powering off when the MCU is ready, or the reset condition is met"
- note added: "TODO: ribbon cable connector"
- moved on the sheet: BT1, D17, D18, R1, R2, U1
