File: hardware/device/rf.kicad_sch (KiCad schematic)
At the start: 7 parts, among them U22 nRF, Y2 32.768kHz

Commit message: feat: clean up footprints, route bluetooth module
Connections:
- net AUDIO_UART.RX: now also PS1.B1 (P0.08/TRACEDATA3/SCK)
- net AUDIO_UART.TX: now also PS1.C1 (P0.10/TRACEDATA1/MISO)
- net BCLK: now also PS1.F1 (P0.17/SCK); no longer PS1.E2 (P0.14/IO1)
- net DACDAT: now also PS1.H1 (P0.24); no longer PS1.D2 (P0.13/IO0)
- net LRCLK: now also PS1.E1 (P0.18/CSN); no longer PS1.F2 (P0.16/IO3)
- net MCLK: now also PS1.G1 (P1.06); no longer PS1.A2 (P0.12/TRACECLK/DCX)
Other:
- moved on the sheet: Y2

Commit message: feat: add SWD connector, route bluetooth, route velocity matrix
Parts:
- U22: footprint Connector_PinHeader_1.27mm:PinHeader_2x05_P1.27mm_Vertical -> pocket_synth:SAMTEC_FTSH-105-01-F-D-K
Changed lines of the file:
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@@
 			)
 		)
-		(property "Footprint" "Connector_PinHeader_1.27mm:PinHeader_2x05_P1.27mm_Vertical"
+		(property "Footprint" "pocket_synth:SAMTEC_FTSH-105-01-F-D-K"
 			(at 29.21 68.58 0)
 			(effects
